File: ADP1612_Boost_Converter.brd (EAGLE design)
At the start: 29 x 22.5 mm, 13 parts, among them U1 ADP1612ARMZ-R7D

Commit message: Add files via upload
Parts:
- removed SJ2: (no value), jumper:SJW
- added SJ5: (no value), jumper:SJW
- C3, C4: device Capacitor_10uF_smd_CAP-0135:CAPC1608X100N -> EEE-1CA100SR_10uF_SMD:CAPAE430X550N
- D1: value BAS40 -> BAT60J; device diode:SOT23 -> diode:SOD323_ST
- moved C2 54.8 mm to (33.0, 78.0), turned to 180 degrees
- moved R2 54.1 mm to (26.9, 78.2), turned to 180 degrees
- moved R1 52.0 mm to (22.0, 75.0), turned to 90 degrees
- moved C4 51.7 mm to (37.7, 79.1), turned to 270 degrees
- moved R3 49.8 mm to (28.7, 81.6), turned to 0 degrees
- moved C1 47.6 mm to (22.4, 71.9)
- moved C3 45.9 mm to (41.1, 73.2)
- moved SJ1 45.7 mm to (43.9, 66.2)
- moved U1 44.8 mm to (28.5, 74.0), turned to 270 degrees
- moved SJ3 39.8 mm to (27.7, 69.0), turned to 0 degrees
- moved L1 36.5 mm to (35.5, 70.6), turned to 270 degrees
- moved D1 34.6 mm to (40.9, 69.1), turned to 180 degrees
Connections:
- removed net N$3 (its old number): D1.1, L1.2, U1.5
- removed net N$6: C4.2, D1.3, R3.2, SJ2.2
- removed net N$8: C3.2, L1.1, SJ1.2, SJ3.3, U1.6
- new net 5VDC: C4.1, D1.C, R3.2, SJ1.2
- new net N$1: C3.1, L1.1, SJ3.3, SJ5.2, U1.6
- new net N$5: D1.A, L1.2, U1.5
- net GND: now also C3.2, C4.2, SJ5.1; no longer C3.1, C4.1, SJ2.1
Routing:
- net N$6: track 34.9 -> 0.00 mm
- net N$8: track 27.7 -> 0.00 mm
- net N$7: track 16.4 -> 0.00 mm
- net N$3 (its old number): track 13.4 -> 0.00 mm
- net N$4: track 8.10 -> 0.00 mm
- net N$3: track 4.86 -> 0.00 mm
- net N$2: track 3.05 -> 0.17 mm
- net N$9: track 4.19 -> 6.02 mm
- added copper zone on layer 1, net 5VDC
- added copper zone on layer 1, net N$1
- added copper zone on layer 1, net N$2
- added copper zone on layer 1, net N$3
- added copper zone on layer 1, net N$4
- added copper zone on layer 1, net N$5
- added copper zone on layer 1, net N$7
Other:
- board size 29 x 22.5 mm -> 28.6 x 24 mm
- board text added: "+"
- board text added: "GND"
- board text added: "Input 1.8VDC"
- board text removed: "Input 4.2VDC"
- board text removed: "ON/OFF Jumper"
